Commit message: Restore restricted Sharpa AA limits and add equal-head-density study

File: assets/urdf/kuka_sharpa_description/iiwa14_left_sharpa_adjusted_restricted.urdf (robot description, URDF)
Before this commit: robot kuka_sharpa, 43 links, 42 joints
Joints:
- joint left_index_MCP_AA: limit lower=-0.3491 upper=0.3491 effort=1.864 velocity=16.07692878 -> lower=-0.03491 upper=0.03491 effort=1.864 velocity=16.07692878
- joint left_middle_MCP_AA: limit lower=-0.3491 upper=0.3491 effort=1.864 velocity=16.07692878 -> lower=-0.03491 upper=0.03491 effort=1.864 velocity=16.07692878
- joint left_pinky_MCP_AA: limit lower=-0.3491 upper=0.3491 effort=1.864 velocity=16.07692878 -> lower=-0.03491 upper=0.03491 effort=1.864 velocity=16.07692878
- joint left_ring_MCP_AA: limit lower=-0.3491 upper=0.3491 effort=1.864 velocity=16.07692878 -> lower=-0.03491 upper=0.03491 effort=1.864 velocity=16.07692878
- joint left_thumb_CMC_AA: limit lower=-0.3491 upper=0.3491 effort=3.3 velocity=11.84076833 -> lower=-0.3491 upper=0.1309 effort=3.3 velocity=11.84076833
